File: Radio_Digi.kicad_pcb (KiCad board)
At the start: 2 copper layers, 57.1 x 38.1 mm, 22 parts, among them J1 Conn_01x03, J10 Conn_01x02, J2 Conn_01x02, J3 Conn_01x03, J4 Conn_01x03, J5 Conn_01x02, J6 Conn_01x02, J7 Conn_01x03, J8 Conn_01x03, J9 Conn_01x02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

Commit message: Adding diagrams
Other:
- board size 57.1 x 38.1 mm -> 57.1 x 38.2 mm
- board text added: "Au To PC"
- board text added: "Au from PC"
- board text added: "Au from Ra"
- board text added: "Au to Ra"
- board text added: "Giga Technology"
- board text added: "PTT"
- board text added: "Radio Digi"
- board text added: "V1.0"
Changed lines of the file:
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@@
     (links 33)
     (no_connects 0)
-    (area 102.477499 54.534999 159.777501 92.785001)
+    (area 99.636 54.534999 163.0365 92.912001)
     (thickness 1.6)
-    (drawings 4)
+    (drawings 24)
     (tracks 107)
     (zones 0)
@@
     (tags "capacitor 0805")
     (attr smd)
-    (fp_text reference C2 (at 0 -1.75 180) (layer F.SilkS)
+    (fp_text reference C2 (at -1.2065 -2.032 180) (layer F.SilkS)
       (effects (font (size 1 1) (thickness 0.15)))
     )
@@
       (effects (font (size 1 1) (thickness 0.15)))
     )
-    (fp_text user %R (at 0 -1.75 180) (layer F.Fab)
+    (fp_text user %R (at -1.2065 -2.032 180) (layer F.Fab)
       (effects (font (size 1 1) (thickness 0.15)))
     )
@@
       (effects (font (size 1 1) (thickness 0.15)))
     )
-    (fp_text value 1N4148 (at 3.175 -0.635 180) (layer F.Fab)
+    (fp_text value 1N4148 (at -0.762 1.8415 270) (layer F.Fab)
       (effects (font (size 1 1) (thickness 0.15)))
     )
@@
     (descr "2-way 5.0mm pitch terminal block, http://www.philmore-datak.com/mc/Page%20197.pdf")
     (tags "screw terminal block")
-    (fp_text reference J2 (at 2.5 -6 270) (layer F.SilkS)
+    (fp_text reference J2 (at 2.667 2.6035 450) (layer F.SilkS)
       (effects (font (size 1 1) (thickness 0.15)))
     )
@@
       (effects (font (size 1 1) (thickness 0.15)))
     )
-    (fp_text value Conn_01x03 (at 2.6035 2.9845 270) (layer F.Fab)
+    (fp_text value Conn_01x03 (at -1.2065 7.493 360) (layer F.Fab)
       (effects (font (size 1 1) (thickness 0.15)))
     )
@@
       (effects (font (size 1 1) (thickness 0.15)))
     )
-    (fp_text value Conn_01x03 (at 2.3495 2.667 270) (layer F.Fab)
+    (fp_text value Conn_01x03 (at -3.1115 6.858 360) (layer F.Fab)
       (effects (font (size 1 1) (thickness 0.15)))
     )
@@
     (descr "2-way 5.0mm pitch terminal block, http://www.philmore-datak.com/mc/Page%20197.pdf")
     (tags "screw terminal block")
-    (fp_text reference J10 (at 2.5 -6 270) (layer F.SilkS)
+    (fp_text reference J10 (at 2.032 2.6035 270) (layer F.SilkS)
       (effects (font (size 1 1) (thickness 0.15)))
     )
@@
     (descr "2-way 5.0mm pitch terminal block, http://www.philmore-datak.com/mc/Page%20197.pdf")
     (tags "screw terminal block")
-    (fp_text reference J6 (at 2.5 -6 270) (layer F.SilkS)
+    (fp_text reference J6 (at 2.667 2.6035 270) (layer F.SilkS)
       (effects (font (size 1 1) (thickness 0.15)))
     )
@@
     )
   )
+  (gr_text "Au from Ra" (at 159.004 86.487 270) (layer F.SilkS)
+    (effects (font (size 1.1 1.1) (thickness 0.275)))
+  )
+  (gr_text "Au to Ra" (at 159.004 75.692 270) (layer F.SilkS)
+    (effects (font (size 1.1 1.1) (thickness 0.275)))
+  )
+  (gr_text "Au To PC" (at 115.189 83.312 270) (layer F.SilkS)
+    (effects (font (size 1.1 1.1) (thickness 0.275)))
+  )
+  (gr_text "Au from PC" (at 115.189 73.152 270) (layer F.SilkS)
+    (effects (font (size 1.1 1.1) (thickness 0.275)))
+  )
+  (gr_text PTT (at 115.189 62.992 270) (layer F.SilkS)
+    (effects (font (size 1.5 1.5) (thickness 0.3)))
+  )
+  (gr_text "Radio Digi" (at 118.364 56.007) (layer F.SilkS)
+    (effects (font (size 1.5 1.5) (thickness 0.3)))
+  )
+  (gr_line (start 141.859 90.297) (end 141.859 92.837) (angle 90) (layer Edge.Cuts) (width 0.15))
+  (gr_line (start 144.399 90.297) (end 141.859 90.297) (angle 90) (layer Edge.Cuts) (width 0.15))
+  (gr_line (start 144.399 92.837) (end 144.399 90.297) (angle 90) (layer Edge.Cuts) (width 0.15))
+  (gr_line (start 144.399 57.277) (end 144.399 54.737) (angle 90) (layer Edge.Cuts) (width 0.15))
+  (gr_line (start 141.859 57.277) (end 144.399 57.277) (angle 90) (layer Edge.Cuts) (width 0.15))
+  (gr_line (start 141.859 54.737) (end 141.859 57.277) (angle 90) (layer Edge.Cuts) (width 0.15))
+  (gr_line (start 110.109 57.277) (end 110.109 54.737) (angle 90) (layer Edge.Cuts) (width 0.15))
+  (gr_line (start 107.569 57.277) (end 110.109 57.277) (angle 90) (layer Edge.Cuts) (width 0.15))
+  (gr_line (start 107.569 54.737) (end 107.569 57.277) (angle 90) (layer Edge.Cuts) (width 0.15))
+  (gr_line (start 110.109 90.297) (end 110.109 92.837) (angle 90) (layer Edge.Cuts) (width 0.15))
+  (gr_line (start 107.569 90.297) (end 110.109 90.297) (angle 90) (layer Edge.Cuts) (width 0.15))
+  (gr_line (start 107.569 92.837) (end 107.569 90.297) (angle 90) (layer Edge.Cuts) (width 0.15))
   (gr_line (start 159.7025 92.71) (end 159.7025 54.61) (angle 90) (layer Edge.Cuts) (width 0.15))
   (gr_line (start 102.5525 92.71) (end 159.7025 92.71) (angle 90) (layer Edge.Cuts) (width 0.15))
   (gr_line (start 102.5525 54.61) (end 102.5525 92.71) (angle 90) (layer Edge.Cuts) (width 0.15))
   (gr_line (start 159.7025 54.61) (end 102.5525 54.61) (angle 90) (layer Edge.Cuts) (width 0.15))
+  (gr_text V1.0 (at 115.189 90.932) (layer F.SilkS)
+    (effects (font (size 1.5 1.5) (thickness 0.3)))
+  )
+  (gr_text "Giga Technology" (at 128.905 91.1225) (layer F.Cu)
+    (effects (font (size 1.5 1.5) (thickness 0.3)))
+  )
   (segment (start 145.7125 77.47) (end 152.0825 77.47) (width 0.75) (layer F.Cu) (net 1))
   (segment (start 152.0825 77.47) (end 153.3525 78.74) (width 0.75) (layer F.Cu) (net 1))
@@
   (segment (start 134.3025 60.96) (end 140.5225 60.96) (width 0.75) (layer F.Cu) (net 7))
   (segment (start 140.5225 60.96) (end 140.6525 60.83) (width 0.75) (layer F.Cu) (net 7))
-  (segment (start 134.3025 63.5) (end 132.0165 63.5) (width 0.75) (layer F.Cu) (net 8))
-  (segment (start 148.5595 58.58) (end 153.3525 58.58) (width 0.75) (layer F.Cu) (net 8))
-  (segment (start 145.9865 56.007) (end 148.5595 58.58) (width 0.75) (layer F.Cu) (net 8))
-  (segment (start 132.08 56.007) (end 145.9865 56.007) (width 0.75) (layer F.Cu) (net 8))
-  (segment (start 131.1275 56.9595) (end 132.08 56.007) (width 0.75) (layer F.Cu) (net 8))
-  (segment (start 131.1275 62.611) (end 131.1275 56.9595) (width 0.75) (layer F.Cu) (net 8))
-  (segment (start 132.0165 63.5) (end 131.1275 62.611) (width 0.75) (layer F.Cu) (net 8))
+  (segment (start 153.3525 58.58) (end 139.352 58.58) (width 0.75) (layer F.Cu) (net 8))
+  (segment (start 131.572 63.5) (end 134.3025 63.5) (width 0.75) (layer F.Cu) (net 8))
+  (segment (start 130.429 62.357) (end 131.572 63.5) (width 0.75) (layer F.Cu) (net 8))
+  (segment (start 130.429 58.547) (end 130.429 62.357) (width 0.75) (layer F.Cu) (net 8))
+  (segment (start 132.969 56.007) (end 130.429 58.547) (width 0.75) (layer F.Cu) (net 8))
+  (segment (start 136.779 56.007) (end 132.969 56.007) (width 0.75) (layer F.Cu) (net 8))
+  (segment (start 139.352 58.58) (end 136.779 56.007) (width 0.75) (layer F.Cu) (net 8))
   (segment (start 140.6525 63.63) (end 134.4325 63.63) (width 0.75) (layer F.Cu) (net 8))
   (segment (start 134.4325 63.63) (end 134.3025 63.5) (width 0.75) (layer F.Cu) (net 8))
